File: kicad-design/6ch-sound-fx-proc/6ch-sound-fx-proc.kicad_pcb (KiCad board)
At the start: 2 copper layers, 59 x 60 mm, 73 parts, among them J1 2.54mm 2-pin, J10 2.54mm 2-pin, J11 2.54mm 2-pin, J12 2.54mm 2-pin, J13 2.54mm 2-pin, J2 2.54mm 2-pin, J3 2.54mm 2-pin, J4 2.54mm 2-pin, J5 2.54mm 2-pin, J6 2.54mm 2-pin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

Commit message: Update version information of the schematic and PCB design.
Other:
- net class Default removed
